File: Issue_4/qdisk_v4.kicad_pcb (KiCad board)
At the start: 2 copper layers, 125.7 x 97.8 mm, 31 parts, among them J1 QL_SLOT_DIN41612_CARD, J2 Conn_02x17_Odd_Even, Q1 PN2222A, U1 7805, U3 LS03, U4 LS11, U6 LS04, U7 LS00, U8 LS240, U9 27C128, Y1 8Mhz

Commit message: initial Issue 3
Parts:
- U10: renamed from U; value FDC_WD1772 -> WD1770
- U11: renamed from U; value 74LS174 -> LS174
- U2: renamed from U; value 74LS266 -> LS266
- U5: renamed from U; value 74LS245 -> LS245
