File: Issue_4/qdisk_v4.kicad_sch (KiCad schematic)
At the start: 31 parts, among them J1 QL_SLOT_DIN41612_CARD, J2 Conn_02x17_Odd_Even, Q1 PN2222A, U1 7805, U3 LS03, U4 LS11, U6 LS04, U7 LS00, U8 LS240, U9 27C128, Y1 8Mhz

Commit message: initial Issue 3
Parts:
- renumbered U to U10, U to U11, U to U2, U to U5
